File: LEDLight/LEDLight.sch (KiCad schematic (older format))
At the start: 18 parts, among them P1 LED Light, P2 PIR Sensor, P3 RF433 Receiver, P4 Light Sensor, P5 INPUT voltage 12V, P6 Thermo drive, Q1 IRLZ44N, Q2 IRLZ44N, U1 arduino_NANO, U2 nRF24L01+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

Commit message: LightSwitch changes
Parts:
- C1, C2: symbol CP_Small -> LEDLight-rescue:CP_Small
- D1, D2: symbol LED -> LEDLight-rescue:LED-RESCUE-LEDLight
- P1, P5, P6: symbol CONN_01X02 -> LEDLight-rescue:CONN_01X02
- P2: symbol CONN_01X03 -> LEDLight-rescue:CONN_01X03
- P3, P4: symbol CONN_01X04 -> LEDLight-rescue:CONN_01X04
- Q1, Q2: symbol IRF540N -> LEDLight-rescue:IRF540N-RESCUE-LEDLight
- R1, R2: symbol R -> LEDLight-rescue:R
- R3: symbol R_Small -> LEDLight-rescue:R_Small
- U1: symbol arduino_mini -> LEDLight-rescue:arduino_mini
- U2: symbol nRF24L01+ -> LEDLight-rescue:nRF24L01+
- U3: symbol DS18B20 -> LEDLight-rescue:DS18B20
Connections:
- wire segments 73 -> 79
Changed lines of the file:
@@
-EESchema Schematic File Version 2
-LIBS:power
-LIBS:device
-LIBS:transistors
-LIBS:conn
-LIBS:linear
-LIBS:regul
-LIBS:74xx
-LIBS:cmos4000
-LIBS:adc-dac
-LIBS:memory
-LIBS:xilinx
-LIBS:microcontrollers
-LIBS:dsp
-LIBS:microchip
-LIBS:analog_switches
-LIBS:motorola
-LIBS:texas
-LIBS:intel
-LIBS:audio
-LIBS:interface
-LIBS:digital-audio
-LIBS:philips
-LIBS:display
-LIBS:cypress
-LIBS:siliconi
-LIBS:opto
-LIBS:atmel
-LIBS:contrib
-LIBS:valves
-LIBS:nRF24L01+
-LIBS:nrf24l01p_smd
-LIBS:arduino
-LIBS:ds18xx
+EESchema Schematic File Version 4
 LIBS:LEDLight-cache
-EELAYER 25 0
+EELAYER 26 0
 EELAYER END
 $Descr A4 11693 8268
@@
 $EndDescr
 $Comp
-L nRF24L01+ U2
+L LEDLight-rescue:nRF24L01+ U2
 U 1 1 5745BE0F
 P 8500 2400
@@
 $EndComp
 $Comp
-L arduino_mini U1
+L LEDLight-rescue:arduino_mini U1
 U 1 1 5745C3A7
 P 6100 3000
@@
 $EndComp
 $Comp
-L GND #PWR01
+L LEDLight-rescue:GND #PWR01
 U 1 1 5745C95A
 P 5150 2050
@@
 $EndComp
 $Comp
-L PWR_FLAG #FLG02
+L LEDLight-rescue:PWR_FLAG #FLG02
 U 1 1 5745C9AB
 P 4500 1600
@@
 $EndComp
 $Comp
-L PWR_FLAG #FLG03
+L LEDLight-rescue:PWR_FLAG #FLG03
 U 1 1 5745C9C3
 P 5150 1600
@@
 $EndComp
 $Comp
-L VCC #PWR04
+L LEDLight-rescue:VCC #PWR04
 U 1 1 5745CB15
 P 4500 2050
@@
 MOSI
 $Comp
-L GND #PWR05
+L LEDLight-rescue:GND #PWR05
 U 1 1 5745D77E
 P 7250 2450
@@
 $EndComp
 $Comp
-L GND #PWR06
+L LEDLight-rescue:GND #PWR06
 U 1 1 5745D810
 P 6100 4700
@@
 NoConn ~ 5400 2600
 $Comp
-L IRF540N Q1
+L LEDLight-rescue:IRF540N-RESCUE-LEDLight Q1
 U 1 1 5745DBB2
 P 8650 4350
@@
 	7650 3300 7650 4400
 $Comp
-L GND #PWR07
+L LEDLight-rescue:GND #PWR07
 U 1 1 5745DCE0
 P 8750 4750
@@
 	8750 4550 8750 4750
 $Comp
-L CONN_01X02 P1
+L LEDLight-rescue:CONN_01X02 P1
 U 1 1 5745DD52
 P 8950 4050
@@
 $EndComp
 $Comp
-L VCC #PWR08
+L LEDLight-rescue:VCC #PWR08
 U 1 1 5745DD9B
 P 8750 3900
@@
 	8750 4100 8750 4150
 $Comp
-L CONN_01X03 P2
+L LEDLight-rescue:CONN_01X03 P2
 U 1 1 5745DFB2
 P 9850 3100
@@
 	9650 3200 9400 3200
 $Comp
-L GND #PWR09
+L LEDLight-rescue:GND #PWR09
 U 1 1 5745E074
 P 9400 3300
@@
 PIRD
 $Comp
-L CONN_01X04 P3
+L LEDLight-rescue:CONN_01X04 P3
 U 1 1 5745EBF6
 P 9850 3800
@@
 $EndComp
 Wire Wire Line
-	9150 3650 9650 3650
-Wire Wire Line
-	9450 3750 9650 3750
+	9150 3650 9250 3650
+Wire Wire Line
+	9450 3750 9600 3750
 Wire Wire Line
 	9650 3850 9600 3850
@@
 Connection ~ 9600 3750
 $Comp
-L GND #PWR010
+L LEDLight-rescue:GND #PWR010
 U 1 1 5745ED28
 P 9450 4050
@@
 $EndComp
 Wire Wire Line
-	9250 3950 9650 3950
+	9250 3950 9450 3950
 Wire Wire Line
 	9450 3950 9450 4050
@@
 RFd
 $Comp
-L CONN_01X04 P4
+L LEDLight-rescue:CONN_01X04 P4
 U 1 1 57460156
 P 9850 4550
@@
 	9650 4600 9450 4600
 $Comp
-L GND #PWR011
+L LEDLight-rescue:GND #PWR011
 U 1 1 57460243
 P 9450 4750
@@
 SCL
 $Comp
-L R R2
+L LEDLight-rescue:R R2
 U 1 1 5746104A
 P 7250 3500
@@
 	6800 3500 7100 3500
 $Comp
-L LED D1
+L LEDLight-rescue:LED-RESCUE-LEDLight D1
 U 1 1 574610FB
 P 7450 3750
@@
 $EndComp
 $Comp
-L GND #PWR012
+L LEDLight-rescue:GND #PWR012
 U 1 1 57461152
 P 7450 4200
@@
 	7450 3950 7450 4200
 $Comp
-L R R1
+L LEDLight-rescue:R R1
 U 1 1 57461213
 P 7150 2950
@@
 $EndComp
 $Comp
-L LED D2
+L LEDLight-rescue:LED-RESCUE-LEDLight D2
 U 1 1 57461262
 P 7600 2950
@@
 $EndComp
 $Comp
-L GND #PWR013
+L LEDLight-rescue:GND #PWR013
 U 1 1 574612A3
 P 7800 3000
@@
 	7300 2950 7400 2950
 $Comp
-L CP_Small C1
+L LEDLight-rescue:CP_Small C1
 U 1 1 57463108
 P 7500 2250
@@
 	7650 2200 7650 2150
 Wire Wire Line
-	7650 2150 7250 2150
+	7650 2150 7500 2150
 Wire Wire Line
 	7250 2150 7250 2450
@@
 	9250 1900 9250 2200
 $Comp
-L CONN_01X02 P5
+L LEDLight-rescue:CONN_01X02 P5
 U 1 1 574698A3
 P 4550 2650
@@
 $EndComp
 $Comp
-L GND #PWR014
+L LEDLight-rescue:GND #PWR014
 U 1 1 57469900
 P 4800 2850
@@
 	6800 2950 7000 2950
 $Comp
-L IRF540N Q2
+L LEDLight-rescue:IRF540N-RESCUE-LEDLight Q2
 U 1 1 57484ED4
 P 8250 3500
@@
 	8050 3250 8050 3550
 $Comp
-L CONN_01X02 P6
+L LEDLight-rescue:CONN_01X02 P6
 U 1 1 57485237
 P 8950 3200
@@
 $EndComp
 $Comp
-L VCC #PWR015
+L LEDLight-rescue:VCC #PWR015
 U 1 1 574852AA
 P 8750 3000
@@
 	8750 3300 8750 3250
 $Comp
-L GND #PWR016
+L LEDLight-rescue:GND #PWR016
 U 1 1 57485381
 P 8350 3850
@@
 	8350 3700 8350 3850
 $Comp
-L CP_Small C2
+L LEDLight-rescue:CP_Small C2
 U 1 1 5749FBF4
 P 9250 3850
@@
 Connection ~ 9450 3950
 $Comp
-L DS18B20 U3
+L LEDLight-rescue:DS18B20 U3
 U 1 1 574A8FCD
 P 7700 5050
@@
 $EndComp
 $Comp
-L GND #PWR017
+L LEDLight-rescue:GND #PWR017
 U 1 1 574A9012
 P 7300 5350
@@
 	7300 4950 7400 4950
 Wire Wire Line
-	7300 4600 7300 4950
+	7300 4600 7300 4750
 Text Label 7300 4700 0    60   ~ 0
 3V3
 Wire Wire Line
-	6800 5050 7400 5050
+	6800 5050 7100 5050
 Wire Wire Line
 	6800 2850 7000 2850
@@
 TEMP
 $Comp
-L R_Small R3
+L LEDLight-rescue:R_Small R3
 U 1 1 574A928B
 P 7100 4850
@@
 Text Label 6850 5050 0    60   ~ 0
 TEMP
+Wire Wire Line
+	9600 3750 9650 3750
+Wire Wire Line
+	7500 2150 7250 2150
+Wire Wire Line
+	9250 3650 9650 3650
+Wire Wire Line
+	9450 3950 9650 3950
+Wire Wire Line
+	7300 4750 7300 4950
+Wire Wire Line
+	7100 5050 7400 5050
 $EndSCHEMATC
