File: Triac/Triac.sch (KiCad schematic (older format))
At the start: 15 parts, among them M1 MOUNTING-HOLE, M2 MOUNTING-HOLE, P1 Control, P2 IN AC230V, P3 OUT AC230V/16A, U1 MOC3041M, U2 BTA16/800BRG

Commit message: LightSwitch changes
Parts:
- D1: symbol LED -> LED-RESCUE-Triac
Changed lines of the file:
@@
 EESchema Schematic File Version 2
+LIBS:Triac-rescue
 LIBS:power
 LIBS:device
@@
 LIBS:contrib
 LIBS:valves
-LIBS:borniers
-LIBS:mounting-hole
-LIBS:hlk-pm01
 LIBS:Triac-cache
 EELAYER 25 0
@@
 $EndComp
 $Comp
-L LED D1
+L LED-RESCUE-Triac D1
 U 1 1 577B781D
 P 4300 1950
